File: hardware/bicore_master_2_slave/neural_network.brd (EAGLE design)
At the start: 119 x 60 mm, 54 parts, among them IC1 74AHC1G14DBV, IC10 74AHC1G14DBV, IC2 74AHC1G14DBV, IC3 74AHC1G14DBV, IC4 74AHC1G14DBV, IC5 74AHC1G14DBV, IC6 74AHC1G14DBV, IC7 74AHC1G14DBV, IC8 74AHC1G14DBV, IC9 74AHC1G14DBV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

Commit message: hw
Parts:
- removed C12, C13: 100n, resistor:C0805
- removed IC10, IC7, IC8, IC9: 74AHC1G14DBV, 74xx-little-de:SOT23-5
- removed R16, R17, R18, R19, R20, R21, R22: 1M, resistor:M0805
- added C14: 22uF, resistor:153CLV-0605
- added SV1, SV2, SV3, SV4: (no value), con-lstb:MA04-1
- added U2: DRV8836, balto:12WSON
- R15: value 1M -> 4k7
- moved R23 84.7 mm to (40.1, 40.7), turned to 270 degrees
- moved U1 79.2 mm to (37.0, 42.0), turned to 180 degrees
- moved R15 58.0 mm to (53.0, 40.7), turned to 270 degrees
- moved C11 46.6 mm to (55.1, 40.7), turned to 270 degrees
- moved C10 45.2 mm to (42.5, 40.7), turned to 270 degrees
- moved C1 6.08 mm to (29.0, 43.0), turned to 90 degrees
- moved C2 6.08 mm to (26.0, 43.0), turned to 90 degrees
- moved C9 6.08 mm to (21.0, 43.0), turned to 270 degrees
- moved D1 5.83 mm to (12.0, 40.0), turned to 180 degrees
Connections:
- removed net N$19: IC8.4
- removed net N$20: C12.2, IC9.2, R17.2, R21.1
- removed net N$21: C12.1
- removed net N$22: IC9.4
- removed net N$23: C13.2, IC10.2, R18.2, R22.1
- removed net N$24: C13.1
- removed net N$25: IC10.4
- removed net N$26: R19.2
- removed net N$27: R20.2
- removed net N$28: R21.2
- removed net N$29: R22.2
- removed net N$35: U1.8
- new net N$30: SV1.4, U1.5
- new net N$31: SV1.3, U1.4
- new net N$33: SV1.2, U1.3
- net B_OUT_0: now also U1.10
- net B_OUT_1: now also U1.9
- net GND: now also C10.2, C11.2, C14.-, SV2.1, SV4.1, U1.11, U2.11, U2.TH; no longer IC10.3, IC7.3, IC8.3, IC9.3, R15.1, R16.1, R17.1, R18.1
- net IN_0: now also SV2.3
- net IN_1: now also SV2.2
- net N$14: now also U2.12; no longer C10.2, IC7.2, R19.1
- net N$15: now also SV3.4, U2.5; no longer C10.1
- net N$16: now also SV3.3, U2.4; no longer IC7.4
- net N$17: now also SV3.2, U2.3; no longer C11.2, IC8.2, R16.2, R20.1
- net N$18: now also SV3.1, U2.2; no longer C11.1
- net N$32: now also U1.12; no longer U1.7, U1.9
- net N$34: now also SV1.1, U1.2; no longer U1.10
- net S0_OUT_0: now also U1.8
- net S0_OUT_1: now also U1.7
- net S1_OUT_0: now also SV4.3, U2.10, U2.8
- net S1_OUT_1: now also SV4.2, U2.7, U2.9
- net VCC: now also C10.1, C11.1, C14.+, R15.1, R23.1, SV2.4, SV4.4, U2.1; no longer IC10.5, IC7.5, IC8.5, IC9.5
Routing:
- net GND: track 0.00 -> 246.8 mm, vias 0 -> 16
- net VCC: track 0.00 -> 97.7 mm, vias 0 -> 3
- net N$1: track 0.00 -> 83.0 mm, vias 0 -> 2
- net B_OUT_1: track 0.00 -> 52.8 mm, vias 0 -> 3
- net B_OUT_0: track 0.00 -> 45.8 mm, vias 0 -> 4
- net S1_OUT_1: track 0.00 -> 32.3 mm, vias 0 -> 1
- net S0_OUT_1: track 0.00 -> 30.6 mm, vias 0 -> 2
- net S1_OUT_0: track 0.00 -> 22.3 mm, vias 0 -> 3
- net S0_OUT_0: track 0.00 -> 21.5 mm, vias 0 -> 2
- net N$2: track 0.00 -> 10.2 mm
- net N$4: track 0.00 -> 9.22 mm
- net IN_0: track 0.00 -> 8.15 mm
- net IN_1: track 0.00 -> 7.46 mm
- net N$10: track 0.00 -> 6.76 mm
- net N$12: track 0.00 -> 6.07 mm
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Other:
- board size 119 x 60 mm -> 56 x 28 mm
- board text added: "B_OUT_0"
- board text added: "B_OUT_1"
- board text added: "S0_OUT_0"
- board text added: "S0_OUT_1"
- board text added: "S1_OUT_0"
- board text added: "S1_OUT_1"
