File: hardware/bicore_master_2_slave/neural_network.sch (EAGLE design)
At the start: 54 parts, among them IC1 74AHC1G14DBV, IC10 74AHC1G14DBV, IC2 74AHC1G14DBV, IC3 74AHC1G14DBV, IC4 74AHC1G14DBV, IC5 74AHC1G14DBV, IC6 74AHC1G14DBV, IC7 74AHC1G14DBV, IC8 74AHC1G14DBV, IC9 74AHC1G14DBV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

Commit message: hw
Parts:
- removed C12, C13: 100n, resistor:C-EUC0805
- removed IC10, IC7, IC8, IC9: 74AHC1G14DBV, 74xx-little-de:74AHC1G14DBV
- removed R16, R17, R18, R19, R20, R21, R22: 1M, resistor:R-EU_M0805
- added C14: 22uF, resistor:CPOL-EU153CLV-0605
- added SV1, SV2, SV3, SV4: (no value), con-lstb:MA04-1
- added U2: DRV8836, balto:DRV8836
- R15: value 1M -> 4k7
Connections:
- removed net N$19: IC8A.O
- removed net N$20: C12.2, IC9A.I, R17.2, R21.1
- removed net N$21: C12.1
- removed net N$22: IC9A.O
- removed net N$23: C13.2, IC10A.I, R18.2, R22.1
- removed net N$24: C13.1
- removed net N$25: IC10A.O
- removed net N$26: R19.2
- removed net N$27: R20.2
- removed net N$28: R21.2
- removed net N$29: R22.2
- removed net N$35: U1.BIN1/BPHASE
- removed net N$36: U1.AOUT1
- removed net N$37: U1.BOUT1
- new net N$30: SV1.4, U1.BOUT2
- new net N$31: SV1.3, U1.BOUT1
- new net N$33: SV1.2, U1.AOUT2
- net B_OUT_0: now also U1.AIN1/PHASE
- net B_OUT_1: now also U1.AIN2/AENBL
- net GND: now also C10.2, C11.2, C14.-, SV2.1, SV4.1, U1.MODE, U2.MODE, U2.TH; no longer R15.1, R16.1, R17.1, R18.1
- net IN_0: now also SV2.3
- net IN_1: now also SV2.2
- net N$14: now also U2.NSLEEP; no longer C10.2, IC7A.I, R19.1
- net N$15: now also SV3.4, U2.BOUT2; no longer C10.1
- net N$16: now also SV3.3, U2.BOUT1; no longer IC7A.O
- net N$17: now also SV3.2, U2.AOUT2; no longer C11.2, IC8A.I, R16.2, R20.1
- net N$18: now also SV3.1, U2.AOUT1; no longer C11.1
- net N$32: now also U1.NSLEEP; no longer U1.AIN2/AENBL, U1.BIN2/BENBL
- net N$34: now also SV1.1, U1.AOUT1; no longer U1.AIN1/PHASE
- net S0_OUT_0: now also U1.BIN1/BPHASE
- net S0_OUT_1: now also U1.BIN2/BENBL
- net S1_OUT_0: now also SV4.3, U2.AIN1/PHASE, U2.BIN1/BPHASE
- net S1_OUT_1: now also SV4.2, U2.AIN2/AENBL, U2.BIN2/BENBL
- net VCC: now also C10.1, C11.1, C14.+, R15.1, R23.1, SV2.4, SV4.4, U2.VCC
Other:
- moved on the sheet: C10, C11, R15
