File: hardware/bicore_master_2_slave/bicore_master_2_slave.sch (EAGLE design)
At the start: 44 parts, among them IC1 74AHC1G14DBV, IC2 74AHC1G14DBV, IC3 74AHC1G14DBV, IC4 74AHC1G14DBV, IC5 74AHC1G14DBV, IC6 74AHC1G14DBV, U1 DRV8836, U2 DRV8836

Commit message: common
Parts:
- added C10, C11: 100n, resistor:C-EUC0805
- added SV4: (no value), con-lstb:MA04-1
- added U$1, U$2, U$3: ADAFRUIT_FIDUCIAL, main_board:ADAFRUIT_FIDUCIAL
Connections:
- net GND: now also C10.2, C11.2, SV4.1
- net S0_OUT_0: no longer U2.BIN1/BPHASE
- net S0_OUT_1: no longer U2.BIN2/BENBL
- net S1_OUT_0: now also SV4.3, U2.BIN1/BPHASE
- net S1_OUT_1: now also SV4.2, U2.BIN2/BENBL
- net VCC: now also C10.1, C11.1, SV4.4
Changed lines of the file:
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@@
 <part name="GND23" library="supply1" library_urn="urn:adsk.eagle:library:371" deviceset="GND" device=""/>
 <part name="SV3" library="con-lstb" library_urn="urn:adsk.eagle:library:162" deviceset="MA04-1" device="" package3d_urn="urn:adsk.eagle:package:8337/1"/>
+<part name="C10" library="resistor" library_urn="urn:adsk.eagle:library:348" deviceset="C-EU" device="C0805" package3d_urn="urn:adsk.eagle:package:26137/1" value="100n"/>
+<part name="C11" library="resistor" library_urn="urn:adsk.eagle:library:348" deviceset="C-EU" device="C0805" package3d_urn="urn:adsk.eagle:package:26137/1" value="100n"/>
+<part name="GND24" library="supply1" library_urn="urn:adsk.eagle:library:371" deviceset="GND" device=""/>
+<part name="GND25" library="supply1" library_urn="urn:adsk.eagle:library:371" deviceset="GND" device=""/>
+<part name="SV4" library="con-lstb" library_urn="urn:adsk.eagle:library:162" deviceset="MA04-1" device="" package3d_urn="urn:adsk.eagle:package:8337/1"/>
+<part name="GND30" library="supply1" library_urn="urn:adsk.eagle:library:371" deviceset="GND" device=""/>
+<part name="P+7" library="supply1" library_urn="urn:adsk.eagle:library:371" deviceset="VCC" device=""/>
+<part name="U$1" library="main_board" deviceset="ADAFRUIT_FIDUCIAL" device=""/>
+<part name="U$2" library="main_board" deviceset="ADAFRUIT_FIDUCIAL" device=""/>
+<part name="U$3" library="main_board" deviceset="ADAFRUIT_FIDUCIAL" device=""/>
 </parts>
 <sheets>
@@
 <instance part="GND23" gate="1" x="276.86" y="86.36" rot="R270"/>
 <instance part="SV3" gate="1" x="342.9" y="96.52" rot="R180"/>
+<instance part="C10" gate="G$1" x="63.5" y="83.82"/>
+<instance part="C11" gate="G$1" x="55.88" y="83.82"/>
+<instance part="GND24" gate="1" x="63.5" y="66.04"/>
+<instance part="GND25" gate="1" x="55.88" y="66.04"/>
+<instance part="SV4" gate="1" x="342.9" y="25.4"/>
+<instance part="GND30" gate="1" x="353.06" y="15.24"/>
+<instance part="P+7" gate="VCC" x="353.06" y="33.02"/>
+<instance part="U$1" gate="G$1" x="88.9" y="149.86"/>
+<instance part="U$2" gate="G$1" x="88.9" y="139.7"/>
+<instance part="U$3" gate="G$1" x="88.9" y="129.54"/>
 </instances>
 <busses>
@@
 <pinref part="GND23" gate="1" pin="GND"/>
 <wire x1="287.02" y1="86.36" x2="279.4" y2="86.36" width="0.1524" layer="91"/>
+</segment>
+<segment>
+<pinref part="C11" gate="G$1" pin="2"/>
+<pinref part="GND25" gate="1" pin="GND"/>
+<wire x1="55.88" y1="78.74" x2="55.88" y2="68.58" width="0.1524" layer="91"/>
+</segment>
+<segment>
+<pinref part="C10" gate="G$1" pin="2"/>
+<pinref part="GND24" gate="1" pin="GND"/>
+<wire x1="63.5" y1="78.74" x2="63.5" y2="68.58" width="0.1524" layer="91"/>
+</segment>
+<segment>
+<pinref part="SV4" gate="1" pin="1"/>
+<wire x1="350.52" y1="20.32" x2="353.06" y2="20.32" width="0.1524" layer="91"/>
+<pinref part="GND30" gate="1" pin="GND"/>
+<wire x1="353.06" y1="20.32" x2="353.06" y2="17.78" width="0.1524" layer="91"/>
 </segment>
 </net>
@@
 <wire x1="71.12" y1="86.36" x2="71.12" y2="96.52" width="0.1524" layer="91"/>
 <junction x="71.12" y="96.52"/>
+<wire x1="71.12" y1="96.52" x2="63.5" y2="96.52" width="0.1524" layer="91"/>
+<pinref part="C11" gate="G$1" pin="1"/>
+<wire x1="63.5" y1="96.52" x2="55.88" y2="96.52" width="0.1524" layer="91"/>
+<wire x1="55.88" y1="96.52" x2="55.88" y2="86.36" width="0.1524" layer="91"/>
+<pinref part="C10" gate="G$1" pin="1"/>
+<wire x1="63.5" y1="86.36" x2="63.5" y2="96.52" width="0.1524" layer="91"/>
+<junction x="63.5" y="96.52"/>
 </segment>
 <segment>
@@
 <pinref part="P+6" gate="VCC" pin="VCC"/>
 <wire x1="281.94" y1="119.38" x2="281.94" y2="121.92" width="0.1524" layer="91"/>
+</segment>
+<segment>
+<pinref part="SV4" gate="1" pin="4"/>
+<wire x1="350.52" y1="27.94" x2="353.06" y2="27.94" width="0.1524" layer="91"/>
+<pinref part="P+7" gate="VCC" pin="VCC"/>
+<wire x1="353.06" y1="27.94" x2="353.06" y2="30.48" width="0.1524" layer="91"/>
 </segment>
 </net>
@@
 <label x="180.34" y="93.98" size="1.778" layer="95" rot="R180"/>
 </segment>
-<segment>
-<pinref part="U2" gate="G$1" pin="BIN1/BPHASE"/>
-<wire x1="287.02" y1="93.98" x2="274.32" y2="93.98" width="0.1524" layer="91"/>
-<label x="271.78" y="93.98" size="1.778" layer="95" rot="R180"/>
-</segment>
 </net>
 <net name="S0_OUT_1" class="0">
@@
 <label x="180.34" y="91.44" size="1.778" layer="95" rot="R180"/>
 </segment>
-<segment>
-<pinref part="U2" gate="G$1" pin="BIN2/BENBL"/>
-<wire x1="287.02" y1="91.44" x2="274.32" y2="91.44" width="0.1524" layer="91"/>
-<label x="271.78" y="91.44" size="1.778" layer="95" rot="R180"/>
-</segment>
 </net>
 <net name="N$10" class="0">
@@
 <label x="271.78" y="101.6" size="1.778" layer="95" rot="R180"/>
 </segment>
+<segment>
+<pinref part="U2" gate="G$1" pin="BIN1/BPHASE"/>
+<wire x1="287.02" y1="93.98" x2="274.32" y2="93.98" width="0.1524" layer="91"/>
+<label x="271.78" y="93.98" size="1.778" layer="95" rot="R180"/>
+</segment>
+<segment>
+<pinref part="SV4" gate="1" pin="3"/>
+<wire x1="350.52" y1="25.4" x2="360.68" y2="25.4" width="0.1524" layer="91"/>
+<label x="363.22" y="25.4" size="1.778" layer="95"/>
+</segment>
 </net>
 <net name="S1_OUT_1" class="0">
@@
 <label x="271.78" y="99.06" size="1.778" layer="95" rot="R180"/>
 </segment>
-</net>
+<segment>
+<pinref part="U2" gate="G$1" pin="BIN2/BENBL"/>
+<wire x1="287.02" y1="91.44" x2="274.32" y2="91.44" width="0.1524" layer="91"/>
+<label x="271.78" y="91.44" size="1.778" layer="95" rot="R180"/>
+</segment>
+<segment>
+<pinref part="SV4" gate="1" pin="2"/>
+<wire x1="350.52" y1="22.86" x2="360.68" y2="22.86" width="0.1524" layer="91"/>
+<label x="363.22" y="22.86" size="1.778" layer="95"/>
+</segment>
+</net>
