File: hardware/delay_line/neural_network.brd (EAGLE design)
At the start: 119 x 60 mm, 54 parts, among them IC1 74AHC1G14DBV, IC10 74AHC1G14DBV, IC2 74AHC1G14DBV, IC3 74AHC1G14DBV, IC4 74AHC1G14DBV, IC5 74AHC1G14DBV, IC6 74AHC1G14DBV, IC7 74AHC1G14DBV, IC8 74AHC1G14DBV, IC9 74AHC1G14DBV, U1 DRV8836

Commit message: hw
Parts:
- removed C5, C6, C7, C8: 100n, resistor:C0805
- removed IC1, IC2, IC3, IC4, IC5, IC6: 74AHC1G14DBV, 74xx-little-de:SOT23-5
- removed LED1, LED2, LED3, LED4, LED5, LED6: (no value), led:SML1206
- removed R1, R11, R12, R13, R14, R3, R5, R7: 1M, resistor:M0805
- removed R10, R2, R4, R6, R8, R9: 4k7, resistor:M0805
- added J1: (no value), SparkFun-Connectors:1X04
- C3: value 100n -> 22uF; device resistor:C0805 -> resistor:153CLV-0605
- moved C4 43.9 mm to (2.00, -15.0)
- moved C3 38.1 mm to (9.00, -6.00)
- moved U1 2.83 mm to (34.0, 44.0), turned to 270 degrees
Connections:
- net N$15 renamed IN
- net N$28 renamed IN_2
- net N$29 renamed IN_3
- removed net B_OUT_0: C4.1, IC1.4, R2.2, R5.2, U1.10
- removed net B_OUT_1: C3.1, IC2.4, R4.2, R7.2, U1.9
- removed net N$10: C7.2, IC5.2, R11.1
- removed net N$11: LED5.A, R9.1
- removed net N$12: C8.2, IC6.2, R12.1
- removed net N$13: LED6.A, R10.1
- removed net N$16: IC7.4
- removed net N$18: C11.1
- removed net N$19: IC8.4
- removed net N$2: C3.2, IC1.2, R1.2, R13.1
- removed net N$21: C12.1
- removed net N$22: IC9.4
- removed net N$24: C13.1
- removed net N$25: IC10.4
- removed net N$26: R19.2
- removed net N$27: R20.2
- removed net N$3: C5.2, IC3.2, R5.1
- removed net N$4: C4.2, IC2.2, R14.1, R3.2
- removed net N$5: LED1.A, R2.1
- removed net N$6: LED3.A, R6.1
- removed net N$7: LED2.A, R4.1
- removed net N$8: C6.2, IC4.2, R7.1
- removed net N$9: LED4.A, R8.1
- removed net S0_OUT_0: IC3.4, R11.2, R6.2, U1.8
- removed net S0_OUT_1: IC4.4, R12.2, R8.2, U1.7
- removed net S1_OUT_0: IC5.4, R9.2
- removed net S1_OUT_1: IC6.4, R10.2
- new net OUT_0: C11.1, IC7.4, U1.10
- new net OUT_1: C12.1, IC8.4, U1.8
- new net OUT_2: C13.1, IC9.4, U1.9
- new net OUT_3: IC10.4, U1.7
- net GND: now also C3.-, C4.2; no longer C5.1, C6.1, C7.1, C8.1, IC1.3, IC2.3, IC3.3, IC4.3, IC5.3, IC6.3, LED1.C, LED2.C, LED3.C, LED4.C, LED5.C, LED6.C, R1.1, R3.1
- net IN_0: now also R19.2; no longer R13.2
- net IN_1: now also R20.2; no longer R14.2
- net N$1: now also IC10.5, IC7.5, IC8.5, IC9.5; no longer IC1.5, IC2.5, IC3.5, IC4.5, IC5.5, IC6.5
- net VCC: now also C3.+, C4.1; no longer IC10.5, IC7.5, IC8.5, IC9.5
