File: hardware/delay_line/neural_network.sch (EAGLE design)
At the start: 52 parts, among them IC1 74AHC1G14DBV, IC10 74AHC1G14DBV, IC2 74AHC1G14DBV, IC3 74AHC1G14DBV, IC4 74AHC1G14DBV, IC5 74AHC1G14DBV, IC6 74AHC1G14DBV, IC7 74AHC1G14DBV, IC8 74AHC1G14DBV, IC9 74AHC1G14DBV

Commit message: hw
Parts:
- removed C5, C6, C7, C8: 100n, resistor:C-EUC0805
- removed IC1, IC2, IC3, IC4, IC5, IC6: 74AHC1G14DBV, 74xx-little-de:74AHC1G14DBV
- removed LED1, LED2, LED3, LED4, LED5, LED6: (no value), led:LEDSML1206
- removed R1, R11, R12, R13, R14, R3, R5, R7: 1M, resistor:R-EU_M0805
- removed R10, R2, R4, R6, R8, R9: 4k7, resistor:R-EU_M0805
- added J1: (no value), SparkFun-Connectors:CONN_04
- added R23: 4k7, resistor:R-EU_M0805
- added U1: DRV8836, balto:DRV8836
- C3: value 100n -> 22uF; device resistor:C-EUC0805 -> resistor:CPOL-EU153CLV-0605
Connections:
- net N$15 renamed IN
- net N$28 renamed IN_2
- net N$29 renamed IN_3
- removed net B_OUT_0: C4.1, IC1A.O, R2.2, R5.2
- removed net B_OUT_1: C3.1, IC2A.O, R4.2, R7.2
- removed net N$10: C7.2, IC5A.I, R11.1
- removed net N$11: LED5.A, R9.1
- removed net N$12: C8.2, IC6A.I, R12.1
- removed net N$13: LED6.A, R10.1
- removed net N$16: IC7A.O
- removed net N$18: C11.1
- removed net N$19: IC8A.O
- removed net N$2: C3.2, IC1A.I, R1.2, R13.1
- removed net N$21: C12.1
- removed net N$22: IC9A.O
- removed net N$24: C13.1
- removed net N$25: IC10A.O
- removed net N$26: R19.2
- removed net N$27: R20.2
- removed net N$3: C5.2, IC3A.I, R5.1
- removed net N$4: C4.2, IC2A.I, R14.1, R3.2
- removed net N$5: LED1.A, R2.1
- removed net N$6: LED3.A, R6.1
- removed net N$7: LED2.A, R4.1
- removed net N$8: C6.2, IC4A.I, R7.1
- removed net N$9: LED4.A, R8.1
- removed net S0_OUT_0: IC3A.O, R11.2, R6.2
- removed net S0_OUT_1: IC4A.O, R12.2, R8.2
- removed net S1_OUT_0: IC5A.O, R9.2
- removed net S1_OUT_1: IC6A.O, R10.2
- new net N$32: R23.2, U1.NSLEEP
- new net N$33: U1.AOUT2
- new net N$36: U1.AOUT1
- new net N$37: U1.BOUT1
- new net N$38: U1.BOUT2
- new net OUT_0: C11.1, IC7A.O, U1.AIN1/PHASE
- new net OUT_1: C12.1, IC8A.O, U1.BIN1/BPHASE
- new net OUT_2: C13.1, IC9A.O, U1.AIN2/AENBL
- new net OUT_3: IC10A.O, U1.BIN2/BENBL
- net GND: now also C3.-, C4.2, IC10P.GND, IC7P.GND, IC8P.GND, IC9P.GND, U1.MODE, U1.TH; no longer C5.1, C6.1, C7.1, C8.1, IC1P.GND, IC2P.GND, IC3P.GND, IC4P.GND, IC5P.GND, IC6P.GND, LED1.C, LED2.C, LED3.C, LED4.C, LED5.C, LED6.C, R1.1, R3.1
- net IN_0: now also R19.2; no longer R13.2
- net IN_1: now also R20.2; no longer R14.2
- net N$1: now also IC10P.VCC, IC7P.VCC, IC8P.VCC, IC9P.VCC; no longer IC1P.VCC, IC2P.VCC, IC3P.VCC, IC4P.VCC, IC5P.VCC, IC6P.VCC
- net VCC: now also C3.+, C4.1, U1.VCC
Other:
- moved on the sheet: C10, C11, C12, C13, C4, IC10, IC7, IC8, IC9, R15, R16, R17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
