File: hardware/delay_line/delay_line.brd (EAGLE design)
At the start: 56 x 28 mm, 47 parts, among them IC1 74AHC1G14DBV, IC2 74AHC1G14DBV, IC3 74AHC1G14DBV, IC4 74AHC1G14DBV, IC5 74AHC1G14DBV, IC6 74AHC1G14DBV, U1 DRV8836, U2 DRV8836

Commit message: common
Parts:
- removed C11, C7, C8: 100n, resistor:C0805
- removed IC5, IC6: 74AHC1G14DBV, 74xx-little-de:SOT23-5
- removed LED5, LED6: (no value), led:SML1206
- removed R11, R12: 1M, resistor:M0805
- removed R15: 4k7, resistor:M0805
- removed SV2, SV3, SV4: (no value), con-lstb:MA04-1
- removed U2: DRV8836, balto:12WSON
- added U$1, U$2, U$3: ADAFRUIT_FIDUCIAL, main_board:ADAFRUIT_FIDUCIAL_1MM
- R10, R9: value 4k7 -> 1M
- moved R9 64.7 mm to (5.18, -13.7), turned to 0 degrees
- moved R10 63.6 mm to (5.18, -20.1), turned to 0 degrees
- moved R5 42.6 mm to (5.18, -0.91), turned to 0 degrees
- moved R7 41.2 mm to (5.18, -7.32), turned to 0 degrees
- moved C5 30.4 mm to (5.18, 11.9)
- moved C6 29.4 mm to (5.18, 5.49)
- moved D1 2.74 mm to (9.26, 40.0)
Connections:
- removed net N$11: LED5.A, R9.1
- removed net N$13: LED6.A, R10.1
- removed net N$14: R15.2, U2.12
- removed net N$15: SV3.4, U2.5
- removed net N$16: SV3.3, U2.4
- removed net N$17: SV3.2, U2.3
- removed net N$18: SV3.1, U2.2
- removed net S1_OUT_0: IC5.4, R9.2, SV4.3, U2.10, U2.8
- removed net S1_OUT_1: IC6.4, R10.2, SV4.2, U2.7, U2.9
- new net IN: C3.1
- net B_OUT_0: now also C5.1; no longer R5.2
- net B_OUT_1: now also C6.1; no longer C3.1, R7.2
- net GND: now also R5.1, R7.1; no longer C11.2, C5.1, C6.1, C7.1, C8.1, IC5.3, IC6.3, LED5.C, LED6.C, SV2.1, SV4.1, U2.11, U2.TH
- net IN_0: no longer SV2.3
- net IN_1: no longer SV2.2
- net N$1: no longer IC5.5, IC6.5
- net N$10: now also R9.2; no longer C7.2, IC5.2, R11.1
- net N$12: now also R10.2; no longer C8.2, IC6.2, R12.1
- net N$3: now also R5.2, R9.1; no longer R5.1
- net N$8: now also R10.1, R7.2; no longer R7.1
- net S0_OUT_0: no longer R11.2
- net S0_OUT_1: no longer R12.2
- net VCC: no longer C11.1, R15.1, SV2.4, SV4.4, U2.1
Routing:
- net GND: track 215.4 -> 0.00 mm, vias 9 -> 0
- net VCC: track 97.7 -> 0.00 mm, vias 3 -> 0
- net B_OUT_1: track 52.8 -> 0.00 mm, vias 3 -> 0
- net N$1: track 52.0 -> 0.00 mm
- net B_OUT_0: track 45.8 -> 0.00 mm, vias 4 -> 0
- net S0_OUT_1: track 30.6 -> 0.00 mm, vias 2 -> 0
- net S0_OUT_0: track 15.3 -> 0.00 mm, vias 1 -> 0
- net N$2: track 10.2 -> 0.00 mm
- net N$4: track 9.22 -> 0.00 mm
- net S1_OUT_1: track 8.58 -> 0.00 mm
- net IN_0: track 8.15 -> 0.00 mm
- net IN_1: track 7.46 -> 0.00 mm
- net S1_OUT_0: track 6.50 -> 0.00 mm, vias 2 -> 0
- net N$15: track 6.06 -> 0.00 mm
- net N$18: track 6.04 -> 0.00 mm
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Other:
- board text added: "B_OUT_0"
- board text added: "B_OUT_1"
- board text added: "GND"
- board text added: "IN_0"
- board text added: "IN_1"
- board text added: "MASTER"
- board text added: "S0_OUT_0"
- board text added: "S0_OUT_1"
- board text added: "S1_OUT_0"
- board text added: "S1_OUT_1"
- board text added: "SLAVE 0"
- board text added: "SLAVE 1"
- board text added: "VCC"

Commit message: board
Parts:
- added SV2, SV3: (no value), con-lstb:MA04-1
- added U$4, U$5, U$6, U$7: SOLDER_PADNOSTOP, JCM:SOLDER_PAD_NOSTOP
- moved R9 57.4 mm to (50.9, 21.0)
- moved R5 48.7 mm to (50.0, 18.3)
- moved R10 47.0 mm to (39.6, 11.9), turned to 180 degrees
- moved C5 45.8 mm to (50.9, 14.6)
- moved R7 41.9 mm to (43.0, 10.7), turned to 90 degrees
- moved C6 34.7 mm to (39.6, 9.45)
- moved IC4 30.2 mm to (58.3, 10.5)
- moved R8 28.4 mm to (60.9, 7.11), turned to 0 degrees
- moved IC3 28.0 mm to (46.7, 10.6)
- moved R6 27.9 mm to (50.0, 6.81), turned to 0 degrees
- moved LED4 27.1 mm to (55.9, 7.15)
- moved U$3 26.5 mm to (12.8, 6.40)
- moved LED3 26.5 mm to (45.0, 6.92)
- moved R2 25.5 mm to (24.7, 6.48), turned to 0 degrees
- moved C4 25.1 mm to (27.5, 9.10)
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Connections:
- removed net B_OUT_0: C4.1, C5.1, IC1.4, R2.2, U1.10
- removed net B_OUT_1: C6.1, IC2.4, R4.2, U1.9
- removed net N$10: R9.2
- removed net N$12: R10.2
- removed net S0_OUT_0: IC3.4, R6.2, U1.8
- removed net S0_OUT_1: IC4.4, R8.2, U1.7
- new net IN_2: R9.2, U$6.SPAD
- new net IN_3: R10.2, U$7.SPAD
- new net OUT_0: C4.1, IC1.4, R2.2, U1.10
- new net OUT_1: C5.1, IC2.4, R4.2, U1.8
- new net OUT_2: C6.1, IC3.4, R6.2, U1.9
- new net OUT_3: IC4.4, R8.2, SV3.2, SV3.3, U1.7
- net GND: now also SV2.4, SV3.4
- net IN: now also SV2.2
- net IN_0: now also U$4.SPAD
- net IN_1: now also U$5.SPAD
- net VCC: now also SV2.1, SV3.1
Routing:
- net GND: track 0.00 -> 7.45 mm
- net N$34: track 0.00 -> 5.62 mm
- net N$30: track 0.00 -> 5.57 mm
- net VCC: track 0.00 -> 5.13 mm
- net N$31: track 0.00 -> 3.53 mm
- net N$33: track 0.00 -> 3.47 mm
- net N$32: track 0.00 -> 2.00 mm
Other:
- board size 56 x 28 mm -> 62.4 x 24.3 mm
- board text removed: "B_OUT_0"
- board text removed: "B_OUT_1"
- board text removed: "GND"
- board text removed: "IN_0"
- board text removed: "IN_1"
- board text removed: "MASTER"
- board text removed: "S0_OUT_0"
- board text removed: "S0_OUT_1"
- board text removed: "S1_OUT_0"
- board text removed: "S1_OUT_1"
- board text removed: "SLAVE 0"
- board text removed: "SLAVE 1"
- board text removed: "VCC"

Commit message: hw
Parts:
- moved U$6 17.4 mm to (39.9, 14.9)
- moved U$7 15.8 mm to (54.6, 15.2)
- moved R9 14.7 mm to (39.6, 11.6), turned to 180 degrees
- moved C5 12.5 mm to (39.6, 9.14)
- moved R10 12.2 mm to (51.8, 11.6)
- moved C6 12.2 mm to (51.8, 9.45)
- moved R7 11.9 mm to (54.9, 10.4)
- moved R5 10.4 mm to (43.3, 10.4), turned to 90 degrees
- moved SV2 0.30 mm to (8.84, 10.1), turned to 270 degrees
- moved SV3 0.30 mm to (65.8, 10.7), turned to 270 degrees
- moved R13 0.09 mm to (14.4, 11.3), turned to 180 degrees
Connections:
- net OUT_0: now also U1.8; no longer U1.10
- net OUT_1: now also U1.10; no longer U1.8
- net OUT_2: now also U1.7; no longer U1.9
- net OUT_3: now also U1.9; no longer U1.7
Routing:
- net GND: track 7.45 -> 106.4 mm, vias 0 -> 4
- net VCC: track 5.13 -> 88.5 mm
- net N$1: track 0.00 -> 69.6 mm, vias 0 -> 3
- net OUT_0: track 0.00 -> 26.6 mm, vias 0 -> 1
- net OUT_1: track 0.00 -> 25.1 mm, vias 0 -> 1
- net OUT_3: track 0.00 -> 14.9 mm
- net N$2: track 0.00 -> 8.35 mm
- net N$4: track 0.00 -> 8.07 mm
- net N$3: track 0.00 -> 7.73 mm
- net N$8: track 0.00 -> 6.84 mm
- net IN_3: track 0.00 -> 6.79 mm
- net OUT_2: track 0.00 -> 5.61 mm
- net IN: track 0.00 -> 5.60 mm
- net IN_0: track 0.00 -> 4.38 mm
- net IN_2: track 0.00 -> 3.87 mm
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