File: hardware/delay_line/delay_line.sch (EAGLE design)
At the start: 22 parts, among them IC10 74AHC1G14DBV, IC7 74AHC1G14DBV, IC8 74AHC1G14DBV, IC9 74AHC1G14DBV, U1 DRV8836

Commit message: common
Parts:
- removed C11, C12, C13: 100n, resistor:C-EUC0805
- removed IC10, IC7, IC8, IC9: 74AHC1G14DBV, 74xx-little-de:74AHC1G14DBV
- removed R15, R16, R17, R18, R19, R20, R21, R22: 1M, resistor:R-EU_M0805
- added C14: 22uF, resistor:CPOL-EU153CLV-0605
- added C3, C4, C5, C6: 100n, resistor:C-EUC0805
- added IC1, IC2, IC3, IC4: 74AHC1G14DBV, 74xx-little-de:74AHC1G14DBV
- added LED1, LED2, LED3, LED4: (no value), led:LEDSML1206
- added R1, R10, R13, R14, R3, R5, R7, R9: 1M, resistor:R-EU_M0805
- added R2, R4, R6, R8: 4k7, resistor:R-EU_M0805
- added SV1: (no value), con-lstb:MA04-1
- added U$1, U$2, U$3: ADAFRUIT_FIDUCIAL, main_board:ADAFRUIT_FIDUCIAL
Connections:
- removed net N$14: C10.2, IC7A.I, R15.2, R19.1
- removed net N$15: C10.1
- removed net N$17: C11.2, IC8A.I, R16.2, R20.1
- removed net N$20: C12.2, IC9A.I, R17.2, R21.1
- removed net N$23: C13.2, IC10A.I, R18.2, R22.1
- removed net N$25: IC10A.O
- removed net N$26: R19.2
- removed net N$27: R20.2
- removed net N$28: R21.2
- removed net N$29: R22.2
- removed net N$36: U1.AOUT1
- removed net N$37: U1.BOUT1
- removed net N$38: U1.BOUT2
- new net IN: C3.1
- new net IN_0: R13.2
- new net IN_1: R14.2
- new net N$10: R9.2
- new net N$12: R10.2
- new net N$2: C3.2, IC1A.I, R1.2, R13.1
- new net N$3: C5.2, IC3A.I, R5.2, R9.1
- new net N$30: SV1.4, U1.BOUT2
- new net N$31: SV1.3, U1.BOUT1
- new net N$34: SV1.1, U1.AOUT1
- new net N$4: C4.2, IC2A.I, R14.1, R3.2
- new net N$5: LED1.A, R2.1
- new net N$6: LED3.A, R6.1
- new net N$7: LED2.A, R4.1
- new net N$8: C6.2, IC4A.I, R10.1, R7.2
- new net N$9: LED4.A, R8.1
- net B_OUT_0: now also C4.1, C5.1, IC1A.O, R2.2
- net B_OUT_1: now also C6.1, IC2A.O, R4.2
- net GND: now also C10.2, C14.-, IC1P.GND, IC2P.GND, IC3P.GND, IC4P.GND, LED1.C, LED2.C, LED3.C, LED4.C, R1.1, R3.1, R5.1, R7.1; no longer IC10P.GND, IC7P.GND, IC8P.GND, IC9P.GND, R15.1, R16.1, R17.1, R18.1
- net N$1: now also IC1P.VCC, IC2P.VCC, IC3P.VCC, IC4P.VCC; no longer IC10P.VCC, IC7P.VCC, IC8P.VCC, IC9P.VCC
- net N$33: now also SV1.2
- net S0_OUT_0: now also IC3A.O, R6.2
- net S0_OUT_1: now also IC4A.O, R8.2
- net VCC: now also C10.1, C14.+, R23.1
Other:
- moved on the sheet: C10

Commit message: board
Parts:
- added SV2, SV3: (no value), con-lstb:MA04-1
- added U$4, U$5, U$6, U$7: SOLDER_PADNOSTOP, JCM:SOLDER_PADNOSTOP
Connections:
- removed net B_OUT_0: C4.1, C5.1, IC1A.O, R2.2, U1.AIN1/PHASE
- removed net B_OUT_1: C6.1, IC2A.O, R4.2, U1.AIN2/AENBL
- removed net N$10: R9.2
- removed net N$12: R10.2
- removed net S0_OUT_0: IC3A.O, R6.2, U1.BIN1/BPHASE
- removed net S0_OUT_1: IC4A.O, R8.2, U1.BIN2/BENBL
- new net IN_2: R9.2, U$6.NET
- new net IN_3: R10.2, U$7.NET
- new net OUT_0: C4.1, IC1A.O, R2.2, U1.AIN1/PHASE
- new net OUT_1: C5.1, IC2A.O, R4.2, U1.BIN1/BPHASE
- new net OUT_2: C6.1, IC3A.O, R6.2, U1.AIN2/AENBL
- new net OUT_3: IC4A.O, R8.2, SV3.2, SV3.3, U1.BIN2/BENBL
- net GND: now also SV2.4, SV3.4
- net IN: now also SV2.2
- net IN_0: now also U$4.NET
- net IN_1: now also U$5.NET
- net VCC: now also SV2.1, SV3.1
Other:
- moved on the sheet: C3, C4, C5, C6, IC1, IC2, IC3, IC4, LED1, LED2, LED3, LED4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

Commit message: hw
Connections:
- net OUT_0: now also U1.BIN1/BPHASE; no longer U1.AIN1/PHASE
- net OUT_1: now also U1.AIN1/PHASE; no longer U1.BIN1/BPHASE
- net OUT_2: now also U1.BIN2/BENBL; no longer U1.AIN2/AENBL
- net OUT_3: now also U1.AIN2/AENBL; no longer U1.BIN2/BENBL
Changed lines of the file:
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@@
 </segment>
 <segment>
-<pinref part="U1" gate="G$1" pin="AIN1/PHASE"/>
-<wire x1="195.58" y1="101.6" x2="182.88" y2="101.6" width="0.1524" layer="91"/>
-<label x="180.34" y="101.6" size="1.778" layer="95" rot="R180"/>
+<pinref part="U1" gate="G$1" pin="BIN1/BPHASE"/>
+<wire x1="195.58" y1="93.98" x2="182.88" y2="93.98" width="0.1524" layer="91"/>
+<label x="180.34" y="93.98" size="1.778" layer="95" rot="R180"/>
 </segment>
 </net>
@@
 </segment>
 <segment>
-<pinref part="U1" gate="G$1" pin="BIN1/BPHASE"/>
-<wire x1="195.58" y1="93.98" x2="182.88" y2="93.98" width="0.1524" layer="91"/>
-<label x="180.34" y="93.98" size="1.778" layer="95" rot="R180"/>
+<pinref part="U1" gate="G$1" pin="AIN1/PHASE"/>
+<wire x1="195.58" y1="101.6" x2="182.88" y2="101.6" width="0.1524" layer="91"/>
+<label x="180.34" y="101.6" size="1.778" layer="95" rot="R180"/>
 </segment>
 </net>
@@
 </segment>
 <segment>
-<pinref part="U1" gate="G$1" pin="AIN2/AENBL"/>
-<wire x1="195.58" y1="99.06" x2="182.88" y2="99.06" width="0.1524" layer="91"/>
-<label x="180.34" y="99.06" size="1.778" layer="95" rot="R180"/>
+<pinref part="U1" gate="G$1" pin="BIN2/BENBL"/>
+<wire x1="195.58" y1="91.44" x2="182.88" y2="91.44" width="0.1524" layer="91"/>
+<label x="180.34" y="91.44" size="1.778" layer="95" rot="R180"/>
 </segment>
 </net>
@@
 </segment>
 <segment>
-<pinref part="U1" gate="G$1" pin="BIN2/BENBL"/>
-<wire x1="195.58" y1="91.44" x2="182.88" y2="91.44" width="0.1524" layer="91"/>
-<label x="180.34" y="91.44" size="1.778" layer="95" rot="R180"/>
-</segment>
-<segment>
 <pinref part="SV3" gate="1" pin="2"/>
 <wire x1="325.12" y1="27.94" x2="322.58" y2="27.94" width="0.1524" layer="91"/>
@@
 <junction x="322.58" y="27.94"/>
 </segment>
+<segment>
+<pinref part="U1" gate="G$1" pin="AIN2/AENBL"/>
+<wire x1="195.58" y1="99.06" x2="182.88" y2="99.06" width="0.1524" layer="91"/>
+<label x="180.34" y="99.06" size="1.778" layer="95" rot="R180"/>
+</segment>
 </net>
