File: hardware/octacore/octacore.brd (EAGLE design)
At the start: 70 x 70 mm, 63 parts, among them IC1 74AC541DW, IC2 74AC541DW, IC3 74AC541DW, IC4 74AC541DW, IC5 74AC541DW

Commit message: octacore
Parts:
- IC1: value 74AC541DW -> 74AC540DW
Changed lines of the file:
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@@
 </autorouter>
 <elements>
-<element name="IC1" library="74xx-eu" library_urn="urn:adsk.eagle:library:85" package="SO20W" package3d_urn="urn:adsk.eagle:package:2018/1" value="74AC541DW" x="35" y="35" rot="R180"/>
+<element name="IC1" library="74xx-eu" library_urn="urn:adsk.eagle:library:85" package="SO20W" package3d_urn="urn:adsk.eagle:package:2018/1" value="74AC540DW" x="35" y="35" rot="R180"/>
 <element name="IC2" library="74xx-eu" library_urn="urn:adsk.eagle:library:85" package="SO20W" package3d_urn="urn:adsk.eagle:package:2018/1" value="74AC541DW" x="55" y="45" rot="R270"/>
 <element name="MOTOR_0" library="main_board" package="JUMPER_JP1" value="" x="65" y="45" smashed="yes" rot="R180">

Commit message: octacore
Parts:
- moved R3 7.02 mm to (37.2, 38.2)
- moved R4 7.02 mm to (35.0, 38.1)
- moved R21 7.00 mm to (32.4, 38.1), turned to 270 degrees
- moved R22 7.00 mm to (30.0, 38.1), turned to 270 degrees
- moved C10 6.34 mm to (37.7, 44.8), turned to 90 degrees
- moved C9 6.31 mm to (35.5, 44.9), turned to 90 degrees
- moved C15 5.80 mm to (29.8, 44.9)
- moved C14 5.80 mm to (32.0, 44.8)
Connections:
- net GND: now also C10.2, C14.2, C15.2, C9.2; no longer R21.2, R22.2, R3.2, R4.2
- net N$11: now also C10.1, R3.2; no longer C9.1, R3.1
- net N$12: now also C9.1, R4.2; no longer C10.1, R4.1
- net N$27: now also C14.1; no longer C14.2
- net N$29: now also C15.1; no longer C15.2
- net N0: now also R3.1; no longer C9.2
- net N1: now also R4.1; no longer C10.2
- net N4: now also R21.2; no longer C14.1
- net N5: now also R22.2; no longer C15.1
Routing:
- net N5: track 77.1 -> 76.1 mm
- net N4: track 63.4 -> 62.5 mm
- net N$12: track 6.78 -> 7.62 mm
- net N1: track 62.4 -> 61.6 mm
- net N$29: track 8.32 -> 7.51 mm
- net N0: track 69.3 -> 68.7 mm
- net GND: vias 21 -> 22
