File: hardware/octacore/octacore.sch (EAGLE design)
At the start: 63 parts, among them IC1 74AC541DW, IC2 74AC541DW, IC3 74AC541DW, IC4 74AC541DW, IC5 74AC541DW

Commit message: octacore
Parts:
- IC1: value 74AC541DW -> 74AC540DW; device 74xx-eu:74AC541DW -> 74xx-eu:74AC540DW
Changed lines of the file:
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@@
 </classes>
 <parts>
-<part name="IC1" library="74xx-eu" library_urn="urn:adsk.eagle:library:85" deviceset="74*541" device="DW" package3d_urn="urn:adsk.eagle:package:2018/1" technology="AC"/>
+<part name="IC1" library="74xx-eu" library_urn="urn:adsk.eagle:library:85" deviceset="74*540" device="DW" package3d_urn="urn:adsk.eagle:package:2018/1" technology="AC"/>
 <part name="IC2" library="74xx-eu" library_urn="urn:adsk.eagle:library:85" deviceset="74*541" device="DW" package3d_urn="urn:adsk.eagle:package:2018/1" technology="AC"/>
 <part name="GND1" library="supply1" library_urn="urn:adsk.eagle:library:371" deviceset="GND" device=""/>

Commit message: octacore
Connections:
- net GND: now also C10.2, C14.2, C15.2, C9.2; no longer R21.2, R22.2, R3.2, R4.2
- net N$11: now also C10.1, R3.2; no longer C9.1, R3.1
- net N$12: now also C9.1, R4.2; no longer C10.1, R4.1
- net N$27: now also C14.1; no longer C14.2
- net N$29: now also C15.1; no longer C15.2
- net N0: now also R3.1; no longer C9.2
- net N1: now also R4.1; no longer C10.2
- net N4: now also R21.2; no longer C14.1
- net N5: now also R22.2; no longer C15.1
Other:
- moved on the sheet: C10, C14, C15, C9, R21, R22, R3, R4
Changed lines of the file:
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@@
 <instance part="GND19" gate="1" x="58.42" y="-96.52"/>
 <instance part="VCC3" gate="G$1" x="58.42" y="-66.04"/>
-<instance part="R3" gate="G$1" x="-66.04" y="50.8" rot="R180"/>
-<instance part="R4" gate="G$1" x="-66.04" y="48.26" rot="R180"/>
+<instance part="R3" gate="G$1" x="-48.26" y="66.04" rot="R270"/>
+<instance part="R4" gate="G$1" x="-53.34" y="66.04" rot="R270"/>
 <instance part="GND20" gate="1" x="-78.74" y="50.8" rot="R270"/>
-<instance part="C9" gate="G$1" x="-55.88" y="55.88" rot="R180"/>
-<instance part="C10" gate="G$1" x="-48.26" y="55.88" rot="R180"/>
+<instance part="C9" gate="G$1" x="-66.04" y="48.26" rot="R270"/>
+<instance part="C10" gate="G$1" x="-60.96" y="50.8" rot="R270"/>
 <instance part="R5" gate="G$1" x="-5.08" y="71.12" rot="R90"/>
 <instance part="R6" gate="G$1" x="-10.16" y="71.12" rot="R90"/>
@@
 <instance part="LED8" gate="G$1" x="269.24" y="2.54" rot="R90"/>
 <instance part="GND29" gate="1" x="281.94" y="2.54" rot="R90"/>
-<instance part="R21" gate="G$1" x="-66.04" y="40.64" rot="R180"/>
-<instance part="R22" gate="G$1" x="-66.04" y="38.1" rot="R180"/>
+<instance part="R21" gate="G$1" x="-55.88" y="30.48" rot="R270"/>
+<instance part="R22" gate="G$1" x="-48.26" y="30.48" rot="R270"/>
 <instance part="GND30" gate="1" x="-78.74" y="40.64" rot="R270"/>
-<instance part="C14" gate="G$1" x="-55.88" y="30.48" rot="R180"/>
-<instance part="C15" gate="G$1" x="-48.26" y="30.48" rot="R180"/>
+<instance part="C14" gate="G$1" x="-60.96" y="40.64" rot="R270"/>
+<instance part="C15" gate="G$1" x="-66.04" y="38.1" rot="R270"/>
 <instance part="R23" gate="G$1" x="-5.08" y="27.94" rot="R90"/>
 <instance part="R24" gate="G$1" x="-10.16" y="27.94" rot="R90"/>
@@
 </segment>
 <segment>
-<pinref part="R3" gate="G$1" pin="2"/>
 <pinref part="GND20" gate="1" pin="GND"/>
-<wire x1="-71.12" y1="50.8" x2="-73.66" y2="50.8" width="0.1524" layer="91"/>
-<pinref part="R4" gate="G$1" pin="2"/>
+<pinref part="C10" gate="G$1" pin="2"/>
+<wire x1="-66.04" y1="50.8" x2="-73.66" y2="50.8" width="0.1524" layer="91"/>
+<pinref part="C9" gate="G$1" pin="2"/>
 <wire x1="-73.66" y1="50.8" x2="-76.2" y2="50.8" width="0.1524" layer="91"/>
 <wire x1="-71.12" y1="48.26" x2="-73.66" y2="48.26" width="0.1524" layer="91"/>
@@
 </segment>
 <segment>
-<pinref part="R22" gate="G$1" pin="2"/>
+<pinref part="GND30" gate="1" pin="GND"/>
+<pinref part="C14" gate="G$1" pin="2"/>
+<wire x1="-66.04" y1="40.64" x2="-73.66" y2="40.64" width="0.1524" layer="91"/>
+<pinref part="C15" gate="G$1" pin="2"/>
+<wire x1="-73.66" y1="40.64" x2="-76.2" y2="40.64" width="0.1524" layer="91"/>
 <wire x1="-71.12" y1="38.1" x2="-73.66" y2="38.1" width="0.1524" layer="91"/>
 <wire x1="-73.66" y1="38.1" x2="-73.66" y2="40.64" width="0.1524" layer="91"/>
-<pinref part="R21" gate="G$1" pin="2"/>
-<wire x1="-73.66" y1="40.64" x2="-71.12" y2="40.64" width="0.1524" layer="91"/>
-<pinref part="GND30" gate="1" pin="GND"/>
-<wire x1="-76.2" y1="40.64" x2="-73.66" y2="40.64" width="0.1524" layer="91"/>
 <junction x="-73.66" y="40.64"/>
 </segment>
@@
 </segment>
 <segment>
-<pinref part="C9" gate="G$1" pin="2"/>
-<wire x1="-55.88" y1="60.96" x2="-55.88" y2="68.58" width="0.1524" layer="91"/>
-<label x="-55.88" y="68.58" size="1.778" layer="95" rot="R90"/>
-</segment>
-<segment>
 <pinref part="R13" gate="G$1" pin="2"/>
 <wire x1="205.74" y1="25.4" x2="200.66" y2="25.4" width="0.1524" layer="91"/>
 <label x="198.12" y="25.4" size="1.778" layer="95" rot="R180"/>
+</segment>
+<segment>
+<pinref part="R3" gate="G$1" pin="1"/>
+<wire x1="-48.26" y1="71.12" x2="-48.26" y2="73.66" width="0.1524" layer="91"/>
+<label x="-48.26" y="76.2" size="1.778" layer="95" rot="R90"/>
 </segment>
 </net>
@@
 </segment>
 <segment>
-<pinref part="C10" gate="G$1" pin="2"/>
-<wire x1="-48.26" y1="60.96" x2="-48.26" y2="68.58" width="0.1524" layer="91"/>
-<label x="-48.26" y="68.58" size="1.778" layer="95" rot="R90"/>
-</segment>
-<segment>
 <pinref part="R14" gate="G$1" pin="2"/>
 <wire x1="205.74" y1="17.78" x2="200.66" y2="17.78" width="0.1524" layer="91"/>
 <label x="198.12" y="17.78" size="1.778" layer="95" rot="R180"/>
+</segment>
+<segment>
+<pinref part="R4" gate="G$1" pin="1"/>
+<wire x1="-53.34" y1="71.12" x2="-53.34" y2="73.66" width="0.1524" layer="91"/>
+<label x="-53.34" y="76.2" size="1.778" layer="95" rot="R90"/>
 </segment>
 </net>
@@
 </segment>
 <segment>
-<pinref part="C14" gate="G$1" pin="1"/>
-<wire x1="-55.88" y1="27.94" x2="-55.88" y2="17.78" width="0.1524" layer="91"/>
-<label x="-55.88" y="15.24" size="1.778" layer="95" rot="R270"/>
+<pinref part="R21" gate="G$1" pin="2"/>
+<wire x1="-55.88" y1="25.4" x2="-55.88" y2="20.32" width="0.1524" layer="91"/>
+<label x="-55.88" y="17.78" size="1.778" layer="95" rot="R270"/>
 </segment>
 </net>
@@
 </segment>
 <segment>
-<pinref part="C15" gate="G$1" pin="1"/>
-<wire x1="-48.26" y1="27.94" x2="-48.26" y2="17.78" width="0.1524" layer="91"/>
-<label x="-48.26" y="15.24" size="1.778" layer="95" rot="R270"/>
+<pinref part="R22" gate="G$1" pin="2"/>
+<wire x1="-48.26" y1="25.4" x2="-48.26" y2="20.32" width="0.1524" layer="91"/>
+<label x="-48.26" y="17.78" size="1.778" layer="95" rot="R270"/>
 </segment>
 </net>
@@
 <segment>
 <pinref part="IC1" gate="A" pin="A3"/>
-<wire x1="-60.96" y1="50.8" x2="-55.88" y2="50.8" width="0.1524" layer="91"/>
-<pinref part="R3" gate="G$1" pin="1"/>
+<wire x1="-58.42" y1="50.8" x2="-48.26" y2="50.8" width="0.1524" layer="91"/>
+<pinref part="C10" gate="G$1" pin="1"/>
+<pinref part="R3" gate="G$1" pin="2"/>
+<wire x1="-48.26" y1="50.8" x2="15.24" y2="50.8" width="0.1524" layer="91"/>
+<wire x1="-48.26" y1="60.96" x2="-48.26" y2="50.8" width="0.1524" layer="91"/>
+<junction x="-48.26" y="50.8"/>
+</segment>
+</net>
+<net name="N$12" class="0">
+<segment>
+<pinref part="IC1" gate="A" pin="A4"/>
+<wire x1="-63.5" y1="48.26" x2="-53.34" y2="48.26" width="0.1524" layer="91"/>
 <pinref part="C9" gate="G$1" pin="1"/>
-<wire x1="-55.88" y1="50.8" x2="15.24" y2="50.8" width="0.1524" layer="91"/>
-<wire x1="-55.88" y1="53.34" x2="-55.88" y2="50.8" width="0.1524" layer="91"/>
-<junction x="-55.88" y="50.8"/>
-</segment>
-</net>
-<net name="N$12" class="0">
-<segment>
-<pinref part="IC1" gate="A" pin="A4"/>
-<wire x1="-60.96" y1="48.26" x2="-48.26" y2="48.26" width="0.1524" layer="91"/>
-<pinref part="R4" gate="G$1" pin="1"/>
-<pinref part="C10" gate="G$1" pin="1"/>
-<wire x1="-48.26" y1="48.26" x2="15.24" y2="48.26" width="0.1524" layer="91"/>
-<wire x1="-48.26" y1="53.34" x2="-48.26" y2="48.26" width="0.1524" layer="91"/>
-<junction x="-48.26" y="48.26"/>
+<pinref part="R4" gate="G$1" pin="2"/>
+<wire x1="-53.34" y1="48.26" x2="15.24" y2="48.26" width="0.1524" layer="91"/>
+<wire x1="-53.34" y1="60.96" x2="-53.34" y2="48.26" width="0.1524" layer="91"/>
+<junction x="-53.34" y="48.26"/>
 </segment>
 </net>
@@
 <segment>
 <pinref part="IC1" gate="A" pin="A7"/>
+<wire x1="15.24" y1="40.64" x2="-55.88" y2="40.64" width="0.1524" layer="91"/>
+<pinref part="C14" gate="G$1" pin="1"/>
 <pinref part="R21" gate="G$1" pin="1"/>
-<wire x1="15.24" y1="40.64" x2="-55.88" y2="40.64" width="0.1524" layer="91"/>
-<pinref part="C14" gate="G$1" pin="2"/>
-<wire x1="-55.88" y1="40.64" x2="-60.96" y2="40.64" width="0.1524" layer="91"/>
+<wire x1="-55.88" y1="40.64" x2="-58.42" y2="40.64" width="0.1524" layer="91"/>
 <wire x1="-55.88" y1="35.56" x2="-55.88" y2="40.64" width="0.1524" layer="91"/>
 <junction x="-55.88" y="40.64"/>
@@
 <net name="N$29" class="0">
 <segment>
+<pinref part="IC1" gate="A" pin="A8"/>
+<wire x1="-63.5" y1="38.1" x2="-48.26" y2="38.1" width="0.1524" layer="91"/>
+<pinref part="C15" gate="G$1" pin="1"/>
 <pinref part="R22" gate="G$1" pin="1"/>
-<pinref part="IC1" gate="A" pin="A8"/>
-<wire x1="-60.96" y1="38.1" x2="-48.26" y2="38.1" width="0.1524" layer="91"/>
-<pinref part="C15" gate="G$1" pin="2"/>
 <wire x1="-48.26" y1="38.1" x2="15.24" y2="38.1" width="0.1524" layer="91"/>
 <wire x1="-48.26" y1="35.56" x2="-48.26" y2="38.1" width="0.1524" layer="91"/>
